File: sch/RP2040-TestPatternGenerator-VGA-Comp.kicad_sch (KiCad schematic)
At the start: 29 parts, among them J1 DE15_Receptacle_HighDensity_M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, J2 CVBS, SW1 SW_Push, SW2 SW_Push, U1 rp2040-zero, U2 AD724JRZ, Y1 3.579545

Commit message: added library files for schematics and footprints for a successful PCB conversion
Parts:
- C1, C2, C3, C4, C5, C6, C7, C8: footprint (none) -> Capacitor_THT:C_Disc_D5.0mm_W2.5mm_P5.00mm
- J2: footprint (none) -> RCA:CUI_RCJ-044
- U1: footprint kleeb:rp2040-zero-smd -> RP2040-Zero:rp2040-zero-smd
- U2: footprint RW_16_ADI -> AD724:RW_16_ADI
- Y1: footprint (none) -> Crystal:Crystal_HC49-4H_Vertical
Changed lines of the file:
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@@
       (effects (font (size 1.27 1.27)))
     )
-    (property "Footprint" "" (at 160.02 105.7148 0)
+    (property "Footprint" "Capacitor_THT:C_Disc_D5.0mm_W2.5mm_P5.00mm" (at 160.02 105.7148 0)
       (effects (font (size 1.27 1.27)) hide)
     )
@@
     (pin "2")
     (instances
-      (project "RP2040-TestPatternGenerator"
+      (project "RP2040-TestPatternGenerator-VGA-Comp"
         (path "/cf6e1f46-c2e8-445c-8dae-9af0be7afdd3"
           (reference "C3") (unit 1)
@@
       (effects (font (size 1.27 1.27)))
     )
-    (property "Footprint" "" (at 160.02 90.4748 0)
+    (property "Footprint" "Capacitor_THT:C_Disc_D5.0mm_W2.5mm_P5.00mm" (at 160.02 90.4748 0)
       (effects (font (size 1.27 1.27)) hide)
     )
@@
     (pin "2")
     (instances
-      (project "RP2040-TestPatternGenerator"
+      (project "RP2040-TestPatternGenerator-VGA-Comp"
         (path "/cf6e1f46-c2e8-445c-8dae-9af0be7afdd3"
           (reference "C1") (unit 1)
@@
       (effects (font (size 1.27 1.27)) (justify left))
     )
-    (property "Footprint" "kleeb:rp2040-zero-smd" (at 49.53 82.55 0)
+    (property "Footprint" "RP2040-Zero:rp2040-zero-smd" (at 49.53 82.55 0)
       (effects (font (size 1.27 1.27)) hide)
     )
@@
     (pin "17")
     (instances
-      (project "RP2040-TestPatternGenerator"
+      (project "RP2040-TestPatternGenerator-VGA-Comp"
         (path "/cf6e1f46-c2e8-445c-8dae-9af0be7afdd3"
           (reference "U1") (unit 1)
@@
     (pin "2")
     (instances
-      (project "RP2040-TestPatternGenerator"
+      (project "RP2040-TestPatternGenerator-VGA-Comp"
         (path "/cf6e1f46-c2e8-445c-8dae-9af0be7afdd3"
           (reference "SW1") (unit 1)
@@
       (effects (font (size 1.27 1.27)))
     )
-    (property "Footprint" "" (at 192.7352 146.05 0)
+    (property "Footprint" "Capacitor_THT:C_Disc_D5.0mm_W2.5mm_P5.00mm" (at 192.7352 146.05 0)
       (effects (font (size 1.27 1.27)) hide)
     )
@@
     (pin "2")
     (instances
-      (project "RP2040-TestPatternGenerator"
+      (project "RP2040-TestPatternGenerator-VGA-Comp"
         (path "/cf6e1f46-c2e8-445c-8dae-9af0be7afdd3"
           (reference "C5") (unit 1)
@@
     (pin "2")
     (instances
-      (project "RP2040-TestPatternGenerator"
+      (project "RP2040-TestPatternGenerator-VGA-Comp"
         (path "/cf6e1f46-c2e8-445c-8dae-9af0be7afdd3"
           (reference "R11") (unit 1)
@@
     (pin "2")
     (instances
-      (project "RP2040-TestPatternGenerator"
+      (project "RP2040-TestPatternGenerator-VGA-Comp"
         (path "/cf6e1f46-c2e8-445c-8dae-9af0be7afdd3"
           (reference "R8") (unit 1)
@@
     (pin "2")
     (instances
-      (project "RP2040-TestPatternGenerator"
+      (project "RP2040-TestPatternGenerator-VGA-Comp"
         (path "/cf6e1f46-c2e8-445c-8dae-9af0be7afdd3"
           (reference "R1") (unit 1)
@@
     (pin "2")
     (instances
-      (project "RP2040-TestPatternGenerator"
+      (project "RP2040-TestPatternGenerator-VGA-Comp"
         (path "/cf6e1f46-c2e8-445c-8dae-9af0be7afdd3"
           (reference "R7") (unit 1)
@@
     (pin "2")
     (instances
-      (project "RP2040-TestPatternGenerator"
+      (project "RP2040-TestPatternGenerator-VGA-Comp"
         (path "/cf6e1f46-c2e8-445c-8dae-9af0be7afdd3"
           (reference "R12") (unit 1)
@@
     (pin "2")
     (instances
-      (project "RP2040-TestPatternGenerator"
+      (project "RP2040-TestPatternGenerator-VGA-Comp"
         (path "/cf6e1f46-c2e8-445c-8dae-9af0be7afdd3"
           (reference "R6") (unit 1)
@@
     (pin "2")
     (instances
-      (project "RP2040-TestPatternGenerator"
+      (project "RP2040-TestPatternGenerator-VGA-Comp"
         (path "/cf6e1f46-c2e8-445c-8dae-9af0be7afdd3"
           (reference "R4") (unit 1)
@@
     (pin "2")
     (instances
-      (project "RP2040-TestPatternGenerator"
+      (project "RP2040-TestPatternGenerator-VGA-Comp"
         (path "/cf6e1f46-c2e8-445c-8dae-9af0be7afdd3"
           (reference "R13") (unit 1)
@@
     (pin "2")
     (instances
-      (project "RP2040-TestPatternGenerator"
+      (project "RP2040-TestPatternGenerator-VGA-Comp"
         (path "/cf6e1f46-c2e8-445c-8dae-9af0be7afdd3"
           (reference "R9") (unit 1)
@@
     (pin "2")
     (instances
-      (project "RP2040-TestPatternGenerator"
+      (project "RP2040-TestPatternGenerator-VGA-Comp"
         (path "/cf6e1f46-c2e8-445c-8dae-9af0be7afdd3"
           (reference "SW2") (unit 1)
@@
       (effects (font (size 1.27 1.27)))
     )
-    (property "Footprint" "" (at 181.3052 146.05 0)
+    (property "Footprint" "Capacitor_THT:C_Disc_D5.0mm_W2.5mm_P5.00mm" (at 181.3052 146.05 0)
       (effects (font (size 1.27 1.27)) hide)
     )
@@
     (pin "2")
     (instances
-      (project "RP2040-TestPatternGenerator"
+      (project "RP2040-TestPatternGenerator-VGA-Comp"
         (path "/cf6e1f46-c2e8-445c-8dae-9af0be7afdd3"
           (reference "C4") (unit 1)
@@
       (effects (font (size 1.524 1.524)))
     )
-    (property "Footprint" "RW_16_ADI" (at 172.72 86.36 0)
+    (property "Footprint" "AD724:RW_16_ADI" (at 172.72 86.36 0)
       (effects (font (size 1.27 1.27) italic) hide)
     )
@@
     (pin "14")
     (instances
-      (project "RP2040-TestPatternGenerator"
+      (project "RP2040-TestPatternGenerator-VGA-Comp"
         (path "/cf6e1f46-c2e8-445c-8dae-9af0be7afdd3"
           (reference "U2") (unit 1)
@@
     (pin "11")
     (instances
-      (project "RP2040-TestPatternGenerator"
+      (project "RP2040-TestPatternGenerator-VGA-Comp"
         (path "/cf6e1f46-c2e8-445c-8dae-9af0be7afdd3"
           (reference "J1") (unit 1)
@@
       (effects (font (size 1.27 1.27)) (justify left))
     )
-    (property "Footprint" "" (at 204.1652 146.05 0)
+    (property "Footprint" "Capacitor_THT:C_Disc_D5.0mm_W2.5mm_P5.00mm" (at 204.1652 146.05 0)
       (effects (font (size 1.27 1.27)) hide)
     )
@@
     (pin "2")
     (instances
-      (project "RP2040-TestPatternGenerator"
+      (project "RP2040-TestPatternGenerator-VGA-Comp"
         (path "/cf6e1f46-c2e8-445c-8dae-9af0be7afdd3"
           (reference "C6") (unit 1)
@@
     (pin "2")
     (instances
-      (project "RP2040-TestPatternGenerator"
+      (project "RP2040-TestPatternGenerator-VGA-Comp"
         (path "/cf6e1f46-c2e8-445c-8dae-9af0be7afdd3"
           (reference "R2") (unit 1)
@@
       (effects (font (size 1.27 1.27)))
     )
-    (property "Footprint" "" (at 167.64 77.1652 0)
+    (property "Footprint" "Capacitor_THT:C_Disc_D5.0mm_W2.5mm_P5.00mm" (at 167.64 77.1652 0)
       (effects (font (size 1.27 1.27)) hide)
     )
@@
     (pin "2")
     (instances
-      (project "RP2040-TestPatternGenerator"
+      (project "RP2040-TestPatternGenerator-VGA-Comp"
         (path "/cf6e1f46-c2e8-445c-8dae-9af0be7afdd3"
           (reference "C7") (unit 1)
@@
       (effects (font (size 1.27 1.27)))
     )
-    (property "Footprint" "" (at 240.03 110.1852 0)
+    (property "Footprint" "Capacitor_THT:C_Disc_D5.0mm_W2.5mm_P5.00mm" (at 240.03 110.1852 0)
       (effects (font (size 1.27 1.27)) hide)
     )
@@
     (pin "2")
     (instances
-      (project "RP2040-TestPatternGenerator"
+      (project "RP2040-TestPatternGenerator-VGA-Comp"
         (path "/cf6e1f46-c2e8-445c-8dae-9af0be7afdd3"
           (reference "C8") (unit 1)
@@
     (pin "2")
     (instances
-      (project "RP2040-TestPatternGenerator"
+      (project "RP2040-TestPatternGenerator-VGA-Comp"
         (path "/cf6e1f46-c2e8-445c-8dae-9af0be7afdd3"
           (reference "D1") (unit 1)
@@
       (effects (font (size 1.27 1.27)))
     )
-    (property "Footprint" "" (at 160.02 98.0948 0)
+    (property "Footprint" "Capacitor_THT:C_Disc_D5.0mm_W2.5mm_P5.00mm" (at 160.02 98.0948 0)
       (effects (font (size 1.27 1.27)) hide)
     )
@@
     (pin "2")
     (instances
-      (project "RP2040-TestPatternGenerator"
+      (project "RP2040-TestPatternGenerator-VGA-Comp"
         (path "/cf6e1f46-c2e8-445c-8dae-9af0be7afdd3"
           (reference "C2") (unit 1)
@@
     (pin "2")
     (instances
-      (project "RP2040-TestPatternGenerator"
+      (project "RP2040-TestPatternGenerator-VGA-Comp"
         (path "/cf6e1f46-c2e8-445c-8dae-9af0be7afdd3"
           (reference "R3") (unit 1)
@@
       (effects (font (size 1.27 1.27)) (justify left))
     )
-    (property "Footprint" "" (at 259.08 109.22 0)
+    (property "Footprint" "RCA:CUI_RCJ-044" (at 259.08 109.22 0)
       (effects (font (size 1.27 1.27)) hide)
     )
@@
     (pin "2")
     (instances
-      (project "RP2040-TestPatternGenerator"
+      (project "RP2040-TestPatternGenerator-VGA-Comp"
         (path "/cf6e1f46-c2e8-445c-8dae-9af0be7afdd3"
           (reference "J2") (unit 1)
@@
     (pin "2")
     (instances
-      (project "RP2040-TestPatternGenerator"
+      (project "RP2040-TestPatternGenerator-VGA-Comp"
         (path "/cf6e1f46-c2e8-445c-8dae-9af0be7afdd3"
           (reference "R5") (unit 1)
@@
       (effects (font (size 1.27 1.27)))
     )
-    (property "Footprint" "" (at 171.45 67.31 0)
+    (property "Footprint" "Crystal:Crystal_HC49-4H_Vertical" (at 171.45 67.31 0)
       (effects (font (size 1.27 1.27)) hide)
     )
@@
     (pin "2")
     (instances
-      (project "RP2040-TestPatternGenerator"
+      (project "RP2040-TestPatternGenerator-VGA-Comp"
         (path "/cf6e1f46-c2e8-445c-8dae-9af0be7afdd3"
           (reference "Y1") (unit 1)
@@
     (pin "2")
     (instances
-      (project "RP2040-TestPatternGenerator"
+      (project "RP2040-TestPatternGenerator-VGA-Comp"
         (path "/cf6e1f46-c2e8-445c-8dae-9af0be7afdd3"
           (reference "R10") (unit 1)

Commit message: first attempt at positioning all components before traces
Parts:
- C6: footprint Capacitor_THT:C_Disc_D5.0mm_W2.5mm_P5.00mm -> Capacitor_THT:CP_Radial_D5.0mm_P2.50mm
- C8: footprint Capacitor_THT:C_Disc_D5.0mm_W2.5mm_P5.00mm -> Capacitor_THT:CP_Radial_D8.0mm_P3.50mm
Changed lines of the file:
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@@
       (effects (font (size 1.27 1.27)) (justify left))
     )
-    (property "Footprint" "Capacitor_THT:C_Disc_D5.0mm_W2.5mm_P5.00mm" (at 204.1652 146.05 0)
+    (property "Footprint" "Capacitor_THT:CP_Radial_D5.0mm_P2.50mm" (at 204.1652 146.05 0)
       (effects (font (size 1.27 1.27)) hide)
     )
@@
       (effects (font (size 1.27 1.27)))
     )
-    (property "Footprint" "Capacitor_THT:C_Disc_D5.0mm_W2.5mm_P5.00mm" (at 240.03 110.1852 0)
+    (property "Footprint" "Capacitor_THT:CP_Radial_D8.0mm_P3.50mm" (at 240.03 110.1852 0)
       (effects (font (size 1.27 1.27)) hide)
     )
